File: maithoga_lcd_board_480x320_R61529.kicad_pcb (KiCad board)
At the start: 2 copper layers, 85 x 54.5 mm, 17 parts, among them P1 Display Connector, P2 LicheePi_Con, P3 TouchXY Connector, U2 DIO5661ST6

Commit message: Generated gerbers
Parts:
- removed P3: TouchXY Connector, Goldpin:Goldpin_4_2_2_54mm_SMT
Connections:
- DIS1 pad P1: (no net) -> 3V3
- DIS1 pad P2: (no net) -> /Display and Touchscreen/TOUCHSCREEN_SDA
- DIS1 pad P3: (no net) -> /Display and Touchscreen/TOUCHSCREEN_SCL
- DIS1 pad P4: (no net) -> /Display and Touchscreen/TOUCHSCREEN_INT
- DIS1 pad P5: (no net) -> /Standard Goldpin Connector/TOUCHSCREEN_RESET
- DIS1 pad P6: (no net) -> GND
- P1 pad 35: (no net) -> /Display and Touchscreen/TOUCHSCREEN_SDA
- P1 pad 36: (no net) -> /Display and Touchscreen/TOUCHSCREEN_SCL
- P1 pad 37: 3V3 -> /Standard Goldpin Connector/TOUCHSCREEN_RESET
- P1 pad 39: (no net) -> /Display and Touchscreen/TOUCHSCREEN_INT
Routing:
- net /Display and Touchscreen/TOUCHSCREEN_SCL: track 0.00 -> 65.8 mm, vias 0 -> 2
- net /Display and Touchscreen/TOUCHSCREEN_INT: track 0.00 -> 56.4 mm, vias 0 -> 2
- net /Display and Touchscreen/TOUCHSCREEN_SDA: track 0.00 -> 53.4 mm, vias 0 -> 2
- net /Standard Goldpin Connector/TOUCHSCREEN_RESET: track 0.00 -> 53.2 mm, vias 0 -> 2
- net /Lichee Pi Display Connector/TPX1: track 43.3 -> 0.00 mm, vias 2 -> 0
- net /Lichee Pi Display Connector/TPY1: track 41.8 -> 0.00 mm, vias 2 -> 0
- net /Lichee Pi Display Connector/TPY2: track 37.6 -> 0.00 mm, vias 1 -> 0
- net /Lichee Pi Display Connector/TPX2: track 34.7 -> 0.00 mm, vias 2 -> 0
- net 3V3: track 149.1 -> 138.2 mm, vias 6 -> 5
- net GND: track 70.3 -> 67.7 mm, vias 57 -> 58
Other:
- rule pad_to_mask_clearance: 0.05 -> 0.07
